File: hardware/kicad/SedentaryDetector.kicad_sch (KiCad schematic)
At the start: 2 parts, among them J1 ESP32-C3_2x9, J2 MPU6050_1x8

Commit message: feat(hardware): ESP32-WROOM-32 2x15 + MPU6050 1x8 PCB layout
PCB (KiCad 10 pcbnew API):
- Board: 80x50mm, centered layout
- J1: ESP32-WROOM-32 2x15 header @ (-30, -17.8)mm
- J2: MPU6050 GY-521 1x8 header @ (30, -7.6)mm
- GND copper pour on B.Cu
- M3 mounting holes at 4 corners
- Net assignments: GND, 3V3, I2C_SDA, I2C_SCL, MPU_INT, VIN_SW

Dimensions: 24.5mm row spacing, 2.54mm pin pitch
Schematics: in KiCad GUI (hand-writing S-expr format is error-prone)
Parts:
- removed J1: ESP32-C3_2x9, Connector_PinHeader_2.54mm:PinHeader_2x09_P2.54mm_Vertical, symbol Connector_Generic:Conn_02x09_Counter_Clockwise
- removed J2: MPU6050_1x8, Connector_PinHeader_2.54mm:PinHeader_1x08_P2.54mm_Vertical, symbol Connector_Generic:Conn_01x08
- added J1: Conn_02x09, symbol Test:J1
Other:
- company: Test -> (none)
- title: Sedentary Detector Carrier Board -> Test
Changed lines of the file:
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@@
-(kicad_sch (version 20230121) (generator eeschema)
-  (paper "A4")
-  (title_block
-    (title "Sedentary Detector Carrier Board")
-    (date "2026-06-20")
-    (rev "v1")
-    (company "Test")
-  )
-  (symbol
-    (lib_id "Connector_Generic:Conn_02x09_Counter_Clockwise")
-    (at 150 100 0)
-    (unit 1)
-    (in_bom yes)
-    (on_board yes)
-    (property "Reference" "J1" (id 0) (at 225.26 133.68 0) (effects (font (size 1.27 1.27)) (justify left bottom)))
-    (property "Value" "ESP32-C3_2x9" (id 1) (at 225.26 128.6 0) (effects (font (size 1.27 1.27)) (justify left bottom)))
-    (property "Footprint" "Connector_PinHeader_2.54mm:PinHeader_2x09_P2.54mm_Vertical" (id 2) (at 225.26 123.52 0) (effects (font (size 1.27 1.27)) (justify left bottom)))
-    (property "Datasheet" "~" (id 3) (at 225.26 118.44 0) (effects (font (size 1.27 1.27)) (justify left bottom)))
-  )
-  (symbol
-    (lib_id "Connector_Generic:Conn_01x08")
-    (at 250 100 0)
-    (unit 1)
-    (in_bom yes)
-    (on_board yes)
-    (property "Reference" "J2" (id 0) (at 300 133.68 0) (effects (font (size 1.27 1.27)) (justify left bottom)))
-    (property "Value" "MPU6050_1x8" (id 1) (at 300 128.6 0) (effects (font (size 1.27 1.27)) (justify left bottom)))
-    (property "Footprint" "Connector_PinHeader_2.54mm:PinHeader_1x08_P2.54mm_Vertical" (id 2) (at 300 123.52 0) (effects (font (size 1.27 1.27)) (justify left bottom)))
-    (property "Datasheet" "~" (id 3) (at 300 118.44 0) (effects (font (size 1.27 1.27)) (justify left bottom)))
-  )
-  (label "GND" (at 125 100 0))
-  (label "3V3" (at 125 102 0))
-  (label "GPIO0" (at 125 104 0))
-  (label "GPIO1" (at 125 106 0))
-  (label "GPIO2" (at 125 108 0))
-  (label "GPIO3" (at 125 110 0))
-  (label "GPIO4" (at 125 112 0))
-  (label "GPIO5" (at 125 114 0))
-  (label "GND" (at 125 116 0))
-  (label "GND" (at 175 100 0))
-  (label "VIN" (at 175 102 0))
-  (label "GPIO6" (at 175 104 0))
-  (label "GPIO7" (at 175 106 0))
-  (label "GPIO8" (at 175 108 0))
-  (label "GPIO9" (at 175 110 0))
-  (label "GPIO10" (at 175 112 0))
-  (label "RX" (at 175 114 0))
-  (label "TX" (at 175 116 0))
-  (label "VCC" (at 275 100 0))
-  (label "GND" (at 275 102 0))
-  (label "SCL" (at 275 104 0))
-  (label "SDA" (at 275 106 0))
-  (label "XDA" (at 275 108 0))
-  (label "XCL" (at 275 110 0))
-  (label "AD0" (at 275 112 0))
-  (label "INT" (at 275 114 0))
-  (wire (pts (xy 125 100) (xy 140 100)))
-  (wire (pts (xy 125 102) (xy 140 102)))
-  (wire (pts (xy 125 104) (xy 140 104)))
-  (wire (pts (xy 125 106) (xy 140 106)))
-  (wire (pts (xy 125 108) (xy 140 108)))
-  (wire (pts (xy 125 110) (xy 140 110)))
-  (wire (pts (xy 125 112) (xy 140 112)))
-  (wire (pts (xy 125 114) (xy 140 114)))
-  (wire (pts (xy 125 116) (xy 140 116)))
-  (wire (pts (xy 175 100) (xy 160 100)))
-  (wire (pts (xy 175 102) (xy 160 102)))
-  (wire (pts (xy 175 104) (xy 160 104)))
-  (wire (pts (xy 175 106) (xy 160 106)))
-  (wire (pts (xy 175 108) (xy 160 108)))
-  (wire (pts (xy 175 110) (xy 160 110)))
-  (wire (pts (xy 175 112) (xy 160 112)))
-  (wire (pts (xy 175 114) (xy 160 114)))
-  (wire (pts (xy 175 116) (xy 160 116)))
-  (wire (pts (xy 275 100) (xy 290 100)))
-  (wire (pts (xy 275 102) (xy 290 102)))
-  (wire (pts (xy 275 104) (xy 290 104)))
-  (wire (pts (xy 275 106) (xy 290 106)))
-  (wire (pts (xy 275 108) (xy 290 108)))
-  (wire (pts (xy 275 110) (xy 290 110)))
-  (wire (pts (xy 275 112) (xy 290 112)))
-  (wire (pts (xy 275 114) (xy 290 114)))
+(kicad_sch (version 20250114) (generator "eeschema")
+	(paper "A4")
+	(title_block
+		(title "Test")
+		(date "2026-06-20")
+	)
+	(symbol (lib_id "Test:J1") (at 50 50 0) (unit 1) (in_bom yes) (on_board yes)
+		(property "Reference" "J1" (at 50 50 0) (effects (font (size 1.27 1.27))))
+		(property "Value" "Conn_02x09" (at 50 47.46 0) (effects (font (size 1.27 1.27))))
+		(property "Footprint" "" (at 50 50 0) (effects (font (size 1.27 1.27)) hide))
+		(property "Datasheet" "" (at 50 50 0) (effects (font (size 1.27 1.27)) hide))
+		(pin "1")
+		(pin "2")
+	)
 )
